Commit message: Update properties_xx.urdf.xacro

File: chuan_nav_ws/src/chuan_bringup/urdf/properties_xx.urdf.xacro (robot description, xacro)
@@ -10,3 +10,6 @@
         <color rgba="1 1 1 0.5"/>
     </material>
+    <material name="fense">
+        <color rgba="0.3 0 0.3 0.8"/>
+    </material>
 </robot>
