Commit message: Update chuan.urdf.xacro

File: chuan_nav_ws/src/chuan_bringup/urdf/chuan.urdf.xacro (robot description, xacro)
@@ -9,5 +9,5 @@
         </visual>
     </link>
-    <link name="laser">
+    <link name="velodyne">
         <visual>
         <geometry>
@@ -17,7 +17,7 @@
         </visual>
     </link>
-    <joint name="laser_to_base_link" type="fixed">
+    <joint name="velodyne_to_base_link" type="fixed">
         <parent link="base_link"/>
-        <child link="laser"/>
+        <child link="velodyne"/>
         <origin rpy="0 0 0" xyz="0.0 0.2 0.18"/>
     </joint>

Commit message: Update chuan.urdf.xacro

File: chuan_nav_ws/src/chuan_bringup/urdf/chuan.urdf.xacro (robot description, xacro)
@@ -4,7 +4,7 @@
         <visual>
         <geometry>
-            <cylinder length="0.1" radius="0.2"/>
+            <box size="1.5 1 0.3"/>
         </geometry>
-        <material name="black"/>
+        <material name="fense"/>
         </visual>
     </link>
@@ -20,5 +20,5 @@
         <parent link="base_link"/>
         <child link="velodyne"/>
-        <origin rpy="0 0 0" xyz="0.0 0.2 0.18"/>
+        <origin rpy="0 0 0" xyz="0.2 0.0 0.5"/>
     </joint>
 </robot>

Commit message: Update chuan.urdf.xacro

File: chuan_nav_ws/src/chuan_bringup/urdf/chuan.urdf.xacro (robot description, xacro)
@@ -4,5 +4,5 @@
         <visual>
         <geometry>
-            <box size="1.5 1 0.3"/>
+            <box size="1.4 1.2 0.7"/>
         </geometry>
         <material name="fense"/>
@@ -12,5 +12,5 @@
         <visual>
         <geometry>
-            <cylinder length="0.05" radius="0.05"/>
+            <cylinder length="0.07" radius="0.05"/>
         </geometry>
         <material name="white"/>
@@ -20,5 +20,5 @@
         <parent link="base_link"/>
         <child link="velodyne"/>
-        <origin rpy="0 0 0" xyz="0.2 0.0 0.5"/>
+        <origin rpy="0 0 0" xyz="0.3 0.0 0.8"/>
     </joint>
 </robot>

Commit message: Update chuan.urdf.xacro

File: chuan_nav_ws/src/chuan_bringup/urdf/chuan.urdf.xacro (robot description, xacro)
@@ -9,5 +9,5 @@
         </visual>
     </link>
-    <link name="velodyne">
+    <link name="laser">
         <visual>
         <geometry>
@@ -17,7 +17,7 @@
         </visual>
     </link>
-    <joint name="velodyne_to_base_link" type="fixed">
+    <joint name="laser_to_base_link" type="fixed">
         <parent link="base_link"/>
-        <child link="velodyne"/>
+        <child link="laser"/>
         <origin rpy="0 0 0" xyz="0.3 0.0 0.8"/>
     </joint>
